Commit message: Add support to connect UR arm to parent platform.
Signed-off-by: Jelmer de Wolde <jelmer.de.wolde@alliander.com>

File: alliander_core/src/alliander_description/ur/urdf/adapted/ur_gz.urdf.xacro (robot description, xacro)
@@ -11,5 +11,5 @@
   <xacro:arg name="name" default="ur"/>
   <!-- import main macro -->
-  <xacro:include filename="$(find ur_description)/urdf/ur_macro.xacro"/>
+  <xacro:include filename="$(find alliander_description)/ur/urdf/adapted/ur_macro.xacro"/>
   <xacro:include filename="$(find alliander_description)/ur/urdf/adapted/ur_gz.ros2_control.xacro" />
   <!-- possible 'ur_type' values: ur3, ur3e, ur5, ur5e, ur7e, ur10, ur10e, ur12e, ur16e, ur8long, ur15, ur18, ur20, ur30 -->
@@ -28,33 +28,10 @@
   <xacro:arg name="simulation_controllers" default="" />
   <xacro:arg name="ros_namespace" default="" />
-  <!-- create link fixed to the "world" -->
-  <link name="world" />
-  <link name="ground_plane">
-    <visual>
-      <origin rpy="0 0 0" xyz="0 0 0"/>
-      <geometry>
-        <box size="5 5 0"/>
-      </geometry>
-      <material name="ground_white">
-        <color rgba="1 1 1 0.5"/>
-      </material>
-    </visual>
-    <collision>
-      <origin rpy="0 0 0" xyz="0 0 0"/>
-      <geometry>
-        <box size="5 5 0"/>
-      </geometry>
-    </collision>
-  </link>
-  <joint name="ground_plane_joint" type="fixed">
-    <origin xyz="0 0 -0.01" rpy="0 0 0"/>
-    <parent link="world"/>
-    <child link="ground_plane"/>
-  </joint>
+  <xacro:arg name="parent" default="world" />
   <!-- arm -->
   <xacro:ur_robot
     name="$(arg name)"
     tf_prefix="$(arg tf_prefix)"
-    parent="world"
+    parent="$(arg parent)"
     joint_limits_parameters_file="$(arg joint_limit_params)"
     kinematics_parameters_file="$(arg kinematics_params)"
