Commit message: Changes so that both simulation and hardware work the same.
Signed-off-by: Jelmer de Wolde <jelmer.de.wolde@alliander.com>

File: alliander_core/src/alliander_description/ewellix/urdf/adapted/ewellix_macro.xacro (robot description, xacro)
@@ -201,6 +201,7 @@
       </joint>
       <link name="${tf_prefix}mount">
-        <inertial>
-          <mass value="0.0001"/> <!-- Gazebo does not spawn the link, when the mass is zero. -->
+        <inertial> <!-- Gazebo does not spawn without inertial link. -->
+          <mass value="0.0001"/>
+          <inertia ixx="0.0001" ixy="0.0" ixz="0.0" iyy="0.0001" iyz="0.0" izz="0.0001"/>
         </inertial>
       </link>
